File: circuit/opamp/opamp.kicad_pcb (KiCad board)
At the start: 2 copper layers, 8 parts, among them J1 Input, J2 Output, J3 Bias Conn, U1 AD711

Commit message: ..
Parts:
- moved J3 30.9 mm to (135.9, 98.8), turned to 90 degrees
- moved R2 8.44 mm to (146.1, 75.7), turned to 180 degrees
- moved J2 6.48 mm to (141.0, 69.8)
- moved C1 3.30 mm to (127.8, 86.6), turned to 90 degrees
- moved J1 2.30 mm to (121.9, 94.2)
- moved C2 1.98 mm to (146.1, 82.3)
- moved R1 1.61 mm to (128.3, 94.2)
Routing:
- net Net-(R1-Pad2): track 0.00 -> 25.4 mm
- net VSS: track 0.00 -> 18.6 mm
- net Net-(J1-Pad1): track 0.00 -> 6.35 mm
Changed lines of the file:
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@@
   (net 9 "Net-(J1-Pad1)")
   (footprint "Connector_PinHeader_2.54mm:PinHeader_1x03_P2.54mm_Vertical" (layer "F.Cu")
-    (at 161.036 80.772)
+    (at 135.905 98.806 90)
     (descr "Through hole straight pin header, 1x03, 2.54mm pitch, single row")
     (tags "Through hole pin header THT 1x03 2.54mm single row")
@@
     (property "Sheetname" "")
     (attr through_hole)
-    (fp_text reference "J3" (at 0 -2.33) (layer "F.SilkS")
-      (effects (font (size 1 1) (thickness 0.15)))
-    )
-    (fp_text value "Bias Conn" (at 0 7.41) (layer "F.Fab")
-      (effects (font (size 1 1) (thickness 0.15)))
-    )
-    (fp_text user "${REFERENCE}" (at 0 2.54 90) (layer "F.Fab")
+    (fp_text reference "J3" (at 0 -2.33 90) (layer "F.SilkS")
+      (effects (font (size 1 1) (thickness 0.15)))
+    )
+    (fp_text value "Bias Conn" (at 0 7.41 90) (layer "F.Fab")
+      (effects (font (size 1 1) (thickness 0.15)))
+    )
+    (fp_text user "${REFERENCE}" (at 0 2.54) (layer "F.Fab")
       (effects (font (size 1 1) (thickness 0.15)))
     )
@@
     (fp_line (start -1.27 -0.635) (end -0.635 -1.27) (layer "F.Fab") (width 0.1))
     (fp_line (start 1.27 -1.27) (end 1.27 6.35) (layer "F.Fab") (width 0.1))
-    (pad "1" thru_hole rect (at 0 0) (size 1.7 1.7) (drill 1) (layers *.Cu *.Mask)
+    (pad "1" thru_hole rect (at 0 0 90) (size 1.7 1.7) (drill 1) (layers *.Cu *.Mask)
       (net 7 "VCC") (pinfunction "Pin_1") (pintype "passive"))
-    (pad "2" thru_hole oval (at 0 2.54) (size 1.7 1.7) (drill 1) (layers *.Cu *.Mask)
+    (pad "2" thru_hole oval (at 0 2.54 90) (size 1.7 1.7) (drill 1) (layers *.Cu *.Mask)
       (net 3 "GND") (pinfunction "Pin_2") (pintype "passive"))
-    (pad "3" thru_hole oval (at 0 5.08) (size 1.7 1.7) (drill 1) (layers *.Cu *.Mask)
+    (pad "3" thru_hole oval (at 0 5.08 90) (size 1.7 1.7) (drill 1) (layers *.Cu *.Mask)
       (net 4 "VSS") (pinfunction "Pin_3") (pintype "passive"))
     (model "${KICAD6_3DMODEL_DIR}/Connector_PinHeader_2.54mm.3dshapes/PinHeader_1x03_P2.54mm_Vertical.wrl"
@@
   )
   (footprint "Capacitor_THT:C_Radial_D5.0mm_H5.0mm_P2.00mm" (layer "F.Cu")
-    (at 147.32 83.82 -90)
+    (at 146.05 82.296 -90)
     (descr "C, Radial series, Radial, pin pitch=2.00mm, diameter=5mm, height=5mm, Non-Polar Electrolytic Capacitor")
     (tags "C Radial series Radial pin pitch 2.00mm diameter 5mm height 5mm Non-Polar Electrolytic Capacitor")
@@
   )
   (footprint "Connector_PinHeader_2.54mm:PinHeader_1x02_P2.54mm_Vertical" (layer "F.Cu")
-    (at 147.32 68.58 90)
+    (at 140.965 69.85 90)
     (descr "Through hole straight pin header, 1x02, 2.54mm pitch, single row")
     (tags "Through hole pin header THT 1x02 2.54mm single row")
@@
   )
   (footprint "Resistor_THT:R_Axial_DIN0207_L6.3mm_D2.5mm_P7.62mm_Horizontal" (layer "F.Cu")
-    (at 137.668 74.676)
+    (at 146.05 75.692 180)
     (descr "Resistor, Axial_DIN0207 series, Axial, Horizontal, pin pitch=7.62mm, 0.25W = 1/4W, length*diameter=6.3*2.5mm^2, http://cdn-reichelt.de/documents/datenblatt/B400/1_4W%23YAG.pdf")
     (tags "Resistor Axial_DIN0207 series Axial Horizontal pin pitch 7.62mm 0.25W = 1/4W length 6.3mm diameter 2.5mm")
@@
     (fp_line (start 6.96 1.25) (end 6.96 -1.25) (layer "F.Fab") (width 0.1))
     (fp_line (start 0.66 -1.25) (end 0.66 1.25) (layer "F.Fab") (width 0.1))
-    (pad "1" thru_hole circle (at 0 0) (size 1.6 1.6) (drill 0.8) (layers *.Cu *.Mask)
+    (pad "1" thru_hole circle (at 0 0 180) (size 1.6 1.6) (drill 0.8) (layers *.Cu *.Mask)
       (net 2 "Net-(R1-Pad2)") (pintype "passive"))
-    (pad "2" thru_hole oval (at 7.62 0) (size 1.6 1.6) (drill 0.8) (layers *.Cu *.Mask)
+    (pad "2" thru_hole oval (at 7.62 0 180) (size 1.6 1.6) (drill 0.8) (layers *.Cu *.Mask)
       (net 6 "Net-(J2-Pad1)") (pintype "passive"))
     (model "${KICAD6_3DMODEL_DIR}/Resistor_THT.3dshapes/R_Axial_DIN0207_L6.3mm_D2.5mm_P7.62mm_Horizontal.wrl"
@@
   )
   (footprint "Connector_PinHeader_2.54mm:PinHeader_1x02_P2.54mm_Vertical" (layer "F.Cu")
-    (at 122.174 91.953 180)
+    (at 121.92 94.239 180)
     (descr "Through hole straight pin header, 1x02, 2.54mm pitch, single row")
     (tags "Through hole pin header THT 1x02 2.54mm single row")
@@
   )
   (footprint "Capacitor_THT:C_Radial_D5.0mm_H5.0mm_P2.00mm" (layer "F.Cu")
-    (at 129.54 83.82 180)
+    (at 127.762 86.598 90)
     (descr "C, Radial series, Radial, pin pitch=2.00mm, diameter=5mm, height=5mm, Non-Polar Electrolytic Capacitor")
     (tags "C Radial series Radial pin pitch 2.00mm diameter 5mm height 5mm Non-Polar Electrolytic Capacitor")
@@
     (property "Sheetname" "")
     (attr through_hole)
-    (fp_text reference "C1" (at 1 -3.75) (layer "F.SilkS")
-      (effects (font (size 1 1) (thickness 0.15)))
-    )
-    (fp_text value "100n" (at 1 3.75) (layer "F.Fab")
-      (effects (font (size 1 1) (thickness 0.15)))
-    )
-    (fp_text user "${REFERENCE}" (at 1 0) (layer "F.Fab")
+    (fp_text reference "C1" (at 1 -3.75 90) (layer "F.SilkS")
+      (effects (font (size 1 1) (thickness 0.15)))
+    )
+    (fp_text value "100n" (at 1 3.75 90) (layer "F.Fab")
+      (effects (font (size 1 1) (thickness 0.15)))
+    )
+    (fp_text user "${REFERENCE}" (at 1 0 90) (layer "F.Fab")
       (effects (font (size 1 1) (thickness 0.15)))
     )
@@
     (fp_circle (center 1 0) (end 3.75 0) (layer "F.CrtYd") (width 0.05) (fill none))
     (fp_circle (center 1 0) (end 3.5 0) (layer "F.Fab") (width 0.1) (fill none))
-    (pad "1" thru_hole circle (at 0 0 180) (size 1.2 1.2) (drill 0.6) (layers *.Cu *.Mask)
+    (pad "1" thru_hole circle (at 0 0 90) (size 1.2 1.2) (drill 0.6) (layers *.Cu *.Mask)
       (net 3 "GND") (pintype "passive"))
-    (pad "2" thru_hole circle (at 2 0 180) (size 1.2 1.2) (drill 0.6) (layers *.Cu *.Mask)
+    (pad "2" thru_hole circle (at 2 0 90) (size 1.2 1.2) (drill 0.6) (layers *.Cu *.Mask)
       (net 7 "VCC") (pintype "passive"))
     (model "${KICAD6_3DMODEL_DIR}/Capacitor_THT.3dshapes/C_Radial_D5.0mm_H5.0mm_P2.00mm.wrl"
@@
   )
   (footprint "Resistor_THT:R_Axial_DIN0207_L6.3mm_D2.5mm_P7.62mm_Horizontal" (layer "F.Cu")
-    (at 128.778 92.71)
+    (at 128.27 94.234)
     (descr "Resistor, Axial_DIN0207 series, Axial, Horizontal, pin pitch=7.62mm, 0.25W = 1/4W, length*diameter=6.3*2.5mm^2, http://cdn-reichelt.de/documents/datenblatt/B400/1_4W%23YAG.pdf")
     (tags "Resistor Axial_DIN0207 series Axial Horizontal pin pitch 7.62mm 0.25W = 1/4W length 6.3mm diameter 2.5mm")
@@
     )
   )
+  (segment (start 135.89 87.63) (end 135.89 94.234) (width 0.762) (layer "F.Cu") (net 2))
+  (segment (start 135.89 83.82) (end 135.89 87.63) (width 0.762) (layer "F.Cu") (net 2))
+  (segment (start 146.05 78.232) (end 140.462 83.82) (width 0.762) (layer "F.Cu") (net 2))
+  (segment (start 140.462 83.82) (end 135.89 83.82) (width 0.762) (layer "F.Cu") (net 2))
+  (segment (start 146.05 75.692) (end 146.05 78.232) (width 0.762) (layer "F.Cu") (net 2))
+  (segment (start 140.97 98.791) (end 140.985 98.806) (width 0.762) (layer "F.Cu") (net 4))
+  (segment (start 144.272 87.63) (end 146.05 85.852) (width 0.762) (layer "F.Cu") (net 4))
+  (segment (start 140.97 87.63) (end 144.272 87.63) (width 0.762) (layer "F.Cu") (net 4))
+  (segment (start 140.97 87.63) (end 140.97 98.791) (width 0.762) (layer "F.Cu") (net 4))
+  (segment (start 146.05 85.852) (end 146.05 84.296) (width 0.762) (layer "F.Cu") (net 4))
+  (segment (start 121.925 94.234) (end 121.92 94.239) (width 0.762) (layer "F.Cu") (net 9))
+  (segment (start 128.27 94.234) (end 121.925 94.234) (width 0.762) (layer "F.Cu") (net 9))
 )

Commit message: ..
Routing:
- net VCC: track 0.00 -> 32.2 mm, vias 0 -> 1
- net Net-(J2-Pad1): track 0.00 -> 11.2 mm
Changed lines of the file:
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@@
   (segment (start 140.97 87.63) (end 140.97 98.791) (width 0.762) (layer "F.Cu") (net 4))
   (segment (start 146.05 85.852) (end 146.05 84.296) (width 0.762) (layer "F.Cu") (net 4))
+  (segment (start 138.43 75.692) (end 138.43 72.385) (width 0.762) (layer "F.Cu") (net 6))
+  (segment (start 138.43 72.385) (end 140.965 69.85) (width 0.762) (layer "F.Cu") (net 6))
+  (segment (start 138.43 80.01) (end 138.43 75.692) (width 0.762) (layer "F.Cu") (net 6))
+  (segment (start 133.35 84.328) (end 133.096 84.582) (width 0.762) (layer "F.Cu") (net 7))
+  (segment (start 135.89 80.01) (end 135.89 81.788) (width 0.762) (layer "F.Cu") (net 7))
+  (segment (start 135.636 82.042) (end 133.35 84.328) (width 0.762) (layer "F.Cu") (net 7))
+  (segment (start 130.048 97.028) (end 130.048 91.44) (width 0.762) (layer "F.Cu") (net 7))
+  (segment (start 135.905 98.806) (end 131.826 98.806) (width 0.762) (layer "F.Cu") (net 7))
+  (segment (start 127.762 84.598) (end 133.08 84.598) (width 0.762) (layer "F.Cu") (net 7))
+  (segment (start 131.826 98.806) (end 130.048 97.028) (width 0.762) (layer "F.Cu") (net 7))
+  (segment (start 135.89 81.788) (end 135.636 82.042) (width 0.762) (layer "F.Cu") (net 7))
+  (segment (start 133.08 84.598) (end 133.35 84.328) (width 0.762) (layer "F.Cu") (net 7))
+  (via (at 130.048 91.44) (size 0.8) (drill 0.4) (layers "F.Cu" "B.Cu") (net 7))
+  (segment (start 130.048 85.598) (end 130.048 91.44) (width 0.762) (layer "B.Cu") (net 7))
+  (segment (start 129.016 84.598) (end 129.032 84.582) (width 0.762) (layer "B.Cu") (net 7))
+  (segment (start 129.032 84.582) (end 130.048 85.598) (width 0.762) (layer "B.Cu") (net 7))
+  (segment (start 127.762 84.598) (end 129.016 84.598) (width 0.762) (layer "B.Cu") (net 7))
   (segment (start 121.925 94.234) (end 121.92 94.239) (width 0.762) (layer "F.Cu") (net 9))
   (segment (start 128.27 94.234) (end 121.925 94.234) (width 0.762) (layer "F.Cu") (net 9))

Commit message: ..
Routing:
- added copper zone on B.Cu, net GND
Changed lines of the file:
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@@
   (segment (start 121.925 94.234) (end 121.92 94.239) (width 0.762) (layer "F.Cu") (net 9))
   (segment (start 128.27 94.234) (end 121.925 94.234) (width 0.762) (layer "F.Cu") (net 9))
+  (zone (net 3) (net_name "GND") (layer "B.Cu") (hatch edge 0.508)
+    (connect_pads (clearance 0.508))
+    (min_thickness 0.254) (filled_areas_thickness no)
+    (fill yes (thermal_gap 0.508) (thermal_bridge_width 0.508))
+    (polygon
+      (pts
+        (xy 155.161657 107.513164)
+        (xy 115.824 107.442)
+        (xy 115.57 64.262)
+        (xy 155.28853 64.249427)
+      )
+    )
+  )
 )

Commit message: ..
Parts:
- moved J3 5.59 mm to (141.5, 98.8)
- moved C2 3.36 mm to (146.6, 85.6)
Routing:
- net VCC: track 32.2 -> 44.9 mm
- net VSS: track 18.6 -> 16.8 mm
Changed lines of the file:
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@@
   (net 9 "Net-(J1-Pad1)")
   (footprint "Connector_PinHeader_2.54mm:PinHeader_1x03_P2.54mm_Vertical" (layer "F.Cu")
-    (at 135.905 98.806 90)
+    (at 141.493 98.806 90)
     (descr "Through hole straight pin header, 1x03, 2.54mm pitch, single row")
     (tags "Through hole pin header THT 1x03 2.54mm single row")
@@
   )
   (footprint "Capacitor_THT:C_Radial_D5.0mm_H5.0mm_P2.00mm" (layer "F.Cu")
-    (at 146.05 82.296 -90)
+    (at 146.558 85.614 -90)
     (descr "C, Radial series, Radial, pin pitch=2.00mm, diameter=5mm, height=5mm, Non-Polar Electrolytic Capacitor")
     (tags "C Radial series Radial pin pitch 2.00mm diameter 5mm height 5mm Non-Polar Electrolytic Capacitor")
@@
   )
   (segment (start 135.89 87.63) (end 135.89 94.234) (width 0.762) (layer "F.Cu") (net 2))
-  (segment (start 135.89 83.82) (end 135.89 87.63) (width 0.762) (layer "F.Cu") (net 2))
-  (segment (start 146.05 78.232) (end 140.462 83.82) (width 0.762) (layer "F.Cu") (net 2))
-  (segment (start 140.462 83.82) (end 135.89 83.82) (width 0.762) (layer "F.Cu") (net 2))
-  (segment (start 146.05 75.692) (end 146.05 78.232) (width 0.762) (layer "F.Cu") (net 2))
-  (segment (start 140.97 98.791) (end 140.985 98.806) (width 0.762) (layer "F.Cu") (net 4))
-  (segment (start 144.272 87.63) (end 146.05 85.852) (width 0.762) (layer "F.Cu") (net 4))
-  (segment (start 140.97 87.63) (end 144.272 87.63) (width 0.762) (layer "F.Cu") (net 4))
-  (segment (start 140.97 87.63) (end 140.97 98.791) (width 0.762) (layer "F.Cu") (net 4))
-  (segment (start 146.05 85.852) (end 146.05 84.296) (width 0.762) (layer "F.Cu") (net 4))
+  (segment (start 135.89 85.598) (end 137.414 84.074) (width 0.762) (layer "F.Cu") (net 2))
+  (segment (start 142.748 84.074) (end 146.05 80.772) (width 0.762) (layer "F.Cu") (net 2))
+  (segment (start 146.05 80.772) (end 146.05 75.692) (width 0.762) (layer "F.Cu") (net 2))
+  (segment (start 137.414 84.074) (end 142.748 84.074) (width 0.762) (layer "F.Cu") (net 2))
+  (segment (start 135.89 87.63) (end 135.89 85.598) (width 0.762) (layer "F.Cu") (net 2))
+  (segment (start 146.558 87.614) (end 140.986 87.614) (width 1.27) (layer "F.Cu") (net 4))
+  (segment (start 146.573 98.806) (end 146.573 87.629) (width 1.27) (layer "F.Cu") (net 4))
+  (segment (start 140.986 87.614) (end 140.97 87.63) (width 1.27) (layer "F.Cu") (net 4))
+  (segment (start 146.573 87.629) (end 146.558 87.614) (width 1.27) (layer "F.Cu") (net 4))
   (segment (start 138.43 75.692) (end 138.43 72.385) (width 0.762) (layer "F.Cu") (net 6))
   (segment (start 138.43 72.385) (end 140.965 69.85) (width 0.762) (layer "F.Cu") (net 6))
   (segment (start 138.43 80.01) (end 138.43 75.692) (width 0.762) (layer "F.Cu") (net 6))
-  (segment (start 133.35 84.328) (end 133.096 84.582) (width 0.762) (layer "F.Cu") (net 7))
-  (segment (start 135.89 80.01) (end 135.89 81.788) (width 0.762) (layer "F.Cu") (net 7))
-  (segment (start 135.636 82.042) (end 133.35 84.328) (width 0.762) (layer "F.Cu") (net 7))
-  (segment (start 130.048 97.028) (end 130.048 91.44) (width 0.762) (layer "F.Cu") (net 7))
-  (segment (start 135.905 98.806) (end 131.826 98.806) (width 0.762) (layer "F.Cu") (net 7))
-  (segment (start 127.762 84.598) (end 133.08 84.598) (width 0.762) (layer "F.Cu") (net 7))
-  (segment (start 131.826 98.806) (end 130.048 97.028) (width 0.762) (layer "F.Cu") (net 7))
-  (segment (start 135.89 81.788) (end 135.636 82.042) (width 0.762) (layer "F.Cu") (net 7))
-  (segment (start 133.08 84.598) (end 133.35 84.328) (width 0.762) (layer "F.Cu") (net 7))
-  (via (at 130.048 91.44) (size 0.8) (drill 0.4) (layers "F.Cu" "B.Cu") (net 7))
-  (segment (start 130.048 85.598) (end 130.048 91.44) (width 0.762) (layer "B.Cu") (net 7))
-  (segment (start 129.016 84.598) (end 129.032 84.582) (width 0.762) (layer "B.Cu") (net 7))
-  (segment (start 129.032 84.582) (end 130.048 85.598) (width 0.762) (layer "B.Cu") (net 7))
-  (segment (start 127.762 84.598) (end 129.016 84.598) (width 0.762) (layer "B.Cu") (net 7))
+  (segment (start 141.493 98.806) (end 134.62 98.806) (width 1.27) (layer "F.Cu") (net 7))
+  (segment (start 132.842 98.806) (end 131.064 97.028) (width 1.27) (layer "F.Cu") (net 7))
+  (segment (start 135.89 80.01) (end 135.89 77.724) (width 1.27) (layer "F.Cu") (net 7))
+  (segment (start 134.112 75.946) (end 129.54 75.946) (width 1.27) (layer "F.Cu") (net 7))
+  (segment (start 127.762 77.724) (end 127.762 84.598) (width 1.27) (layer "F.Cu") (net 7))
+  (segment (start 134.62 98.806) (end 132.842 98.806) (width 1.27) (layer "F.Cu") (net 7))
+  (segment (start 131.064 91.186) (end 131.064 90.424) (width 1.27) (layer "F.Cu") (net 7))
+  (segment (start 129.54 75.946) (end 127.762 77.724) (width 1.27) (layer "F.Cu") (net 7))
+  (segment (start 135.89 77.724) (end 134.112 75.946) (width 1.27) (layer "F.Cu") (net 7))
+  (segment (start 131.064 97.028) (end 131.064 91.186) (width 1.27) (layer "F.Cu") (net 7))
+  (via (at 131.064 90.424) (size 0.8) (drill 0.4) (layers "F.Cu" "B.Cu") (net 7))
+  (segment (start 129.794 84.582) (end 129.778 84.598) (width 1.27) (layer "B.Cu") (net 7))
+  (segment (start 131.064 85.852) (end 129.794 84.582) (width 1.27) (layer "B.Cu") (net 7))
+  (segment (start 131.064 90.424) (end 131.064 85.852) (width 1.27) (layer "B.Cu") (net 7))
+  (segment (start 129.778 84.598) (end 127.762 84.598) (width 1.27) (layer "B.Cu") (net 7))
   (segment (start 121.925 94.234) (end 121.92 94.239) (width 0.762) (layer "F.Cu") (net 9))
   (segment (start 128.27 94.234) (end 121.925 94.234) (width 0.762) (layer "F.Cu") (net 9))

Commit message: ..
Parts:
- C1, C2: footprint Capacitor_THT:C_Radial_D5.0mm_H5.0mm_P2.00mm -> Capacitor_THT:C_Rect_L7.0mm_W2.5mm_P5.00mm
- moved C2 2.06 mm to (146.6, 87.7)
- moved C1 0.48 mm to (127.8, 87.1)
Routing:
- net VCC: track 44.9 -> 51.1 mm
- net VSS: track 16.8 -> 14.9 mm
Other:
- board outline added: 49 x 43.7 mm

Commit message: ..
Other:
- board outline removed
Changed lines of the file:
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@@
     )
   )
-  (gr_rect (start 111.252 63.246) (end 160.274 106.934) (layer "Edge.Cuts") (width 0.1) (fill none))
   (segment (start 135.89 87.63) (end 135.89 94.234) (width 0.762) (layer "F.Cu") (net 2))
   (segment (start 135.89 85.598) (end 137.414 84.074) (width 0.762) (layer "F.Cu") (net 2))
